File: Schematics/KiCad/AirQualityMonitor.kicad_sch (KiCad schematic)
At the start: 9 parts, among them SW1 SW_Push, U2 ESP32-DEVKITC-32E, U3 OLED, U4 BME680, U5 Level Shifter, U7 PMS5003

Commit message: KiCad Files updated
Parts:
- added R2: 5,1k, symbol Device:R
- added U8: DS18B20, symbol _Custom:DS18B20
Connections:
- net at U5. (HV1): now also U2.J3_12 (IO16)
- net at R1.1, U2.J2_1 (3V3), U3.2 (VCC_IN)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: now also R2.1, U8. (GND)
- net at SW1.2, U1. (0V), U2.J3_1 (GND_J3_1)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: now also U8. (GND)
- net at U4. (CS): now also U2.J3_3 (IO22), U3.4 (SDA)
- net at U6. (GND): now also U2.J3_10 (IO5)
- net at U2.J2_11 (IO27): now also R2.2, U8. (GND)
- new net: U1. (0V), U2.J2_19 (EXT_5V), U5. (HV1), U6. (GND), U7.P$8 (VCC)
Other:
- moved on the sheet: U7
