File: Schematics/KiCad/untitled.kicad_sch (KiCad schematic)
At the start: 0 parts

Commit message: KiCad Files updated
Changed lines of the file:
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@@
 	(text "5V+"
 		(exclude_from_sim no)
-		(at 232.156 62.992 0)
+		(at 232.156 56.642 0)
 		(effects
 			(font
@@
 	(text "5V+"
 		(exclude_from_sim no)
-		(at 205.74 113.03 0)
+		(at 205.74 119.38 0)
 		(effects
 			(font
@@
 	(text "Data"
 		(exclude_from_sim no)
-		(at 205.486 116.332 0)
+		(at 205.486 116.078 0)
 		(effects
 			(font
@@
 	(text "GND"
 		(exclude_from_sim no)
-		(at 205.74 119.634 0)
+		(at 205.486 113.03 0)
 		(effects
 			(font
@@
 	(text "Data"
 		(exclude_from_sim no)
-		(at 231.902 56.134 0)
-		(effects
-			(font
+		(at 231.648 62.738 0)
+		(effects
+			(font
